File: mainBoardV3/mainBoardV3.kicad_pcb (KiCad board)
At the start: 2 copper layers, 7 parts, among them J1 Raspberry_Pi_4, U1 Pico

Commit message: Added some progress
Parts:
- added J2: Conn_01x05_Pin, Connector_JST:JST_XH_B5B-XH-A_1x05_P2.50mm_Vertical, F.Cu at (233.1, 116.8)
- added J3: Conn_01x05_Pin, Connector_JST:JST_PH_B5B-PH-K_1x05_P2.00mm_Vertical, F.Cu at (249.5, 144.5)
- added J4: Conn_01x05_Pin, Connector_JST:JST_XH_B5B-XH-A_1x05_P2.50mm_Vertical, F.Cu at (233.1, 124.7)
- added J5: Conn_01x05_Pin, Connector_JST:JST_XH_B5B-XH-A_1x05_P2.50mm_Vertical, F.Cu at (233.1, 132.4)
- added J6: Conn_01x05_Pin, Connector_JST:JST_XH_B5B-XH-A_1x05_P2.50mm_Vertical, F.Cu at (233.1, 140.2)
- added J7: Conn_01x02, Connector_AMASS:AMASS_XT60-M_1x02_P7.20mm_Vertical, F.Cu at (251.7, 118.6)
- added J8: Conn_01x02, Connector_AMASS:AMASS_XT60-F_1x02_P7.20mm_Vertical, F.Cu at (251.7, 128.8)
- added J9: Conn_01x04_Pin, Connector_JST:JST_XH_B4B-XH-A_1x04_P2.50mm_Vertical, F.Cu at (250.0, 137.3)
