File: mainBoardV3/mainBoardV3.kicad_sch (KiCad schematic)
At the start: 16 parts, among them J1 Raspberry_Pi_4, J2 Conn_01x05_Pin, J3 Conn_01x05_Pin, J4 Conn_01x05_Pin, J5 Conn_01x05_Pin, J6 Conn_01x05_Pin, J7 Conn_01x02, J8 Conn_01x02, U1 Pico

Commit message: Added some progress
Parts:
- removed J3: Conn_01x05_Pin, Connector_JST:JST_PH_B5B-PH-K_1x05_P2.00mm_Vertical, symbol Connector:Conn_01x05_Pin
- removed J6: Conn_01x05_Pin, Connector_JST:JST_XH_B5B-XH-A_1x05_P2.50mm_Vertical, symbol Connector:Conn_01x05_Pin
- added C1, C2, C3: 100uF, Capacitor_THT:C_Radial_D6.3mm_H11.0mm_P2.50mm, symbol Device:C_Polarized
- added Stepper1, Stepper2, Stepper3: Conn_01x04_Pin, Connector_JST:JST_XH_B4B-XH-A_1x04_P2.50mm_Vertical, symbol Connector:Conn_01x04_Pin
- added U2: Pico, Ensmasteel_librairy:RPi_Pico_SMD_TH, symbol ENSMASTEEL_librairy:Pico
Connections:
- net GND: now reaches A1.1 (GND)
- net GND: now also A1.7 (GND), A2.1 (GND), A2.7 (GND), A3.1 (GND), A3.7 (GND), C1.2, C2.2, C3.2
- net Stepper1_step: now reaches A1.15 (STEP)
- net Stepper1_dir: now reaches A1.16 (DIR)
- net at A1.3 (A2): now also Stepper1.3 (Pin_3)
- net at A1.4 (A1): now also Stepper1.4 (Pin_4)
- net at A1.5 (B1): now also Stepper1.2 (Pin_2)
- net at A1.6 (B2): now also Stepper1.1 (Pin_1)
- net FusedProtectedVbatt: now reaches A1.8 (VMOT)
- net FusedProtectedVbatt: now also A2.8 (VMOT), A3.8 (VMOT), C1.1, C2.1, C3.1
- net Steppers_en: now reaches A1.9 (~{EN})
- net Steppers_en: now also A2.9 (~{EN}), A3.9 (~{EN})
- net Stepper3_step: now reaches A3.15 (STEP)
- net Stepper3_dir: now reaches A3.16 (DIR)
- net at A3.3 (A2): now also Stepper3.3 (Pin_3)
- net at A3.4 (A1): now also Stepper3.4 (Pin_4)
- net at A3.5 (B1): now also Stepper3.2 (Pin_2)
- net at A3.6 (B2): now also Stepper3.1 (Pin_1)
- net Stepper2_step: now reaches A2.15 (STEP)
- net Stepper2_dir: now reaches A2.16 (DIR)
- net at A2.3 (A2): now also Stepper2.3 (Pin_3)
- net at A2.4 (A1): now also Stepper2.4 (Pin_4)
- net at A2.5 (B1): now also Stepper2.2 (Pin_2)
- net at A2.6 (B2): now also Stepper2.1 (Pin_1)
Other:
- note added: "FOR BIG BOTTOM CONNECTOR"
- note added: "VIO needs to only be on when VBAT is on as to not backfeed voltage to the microcontroller, needs to check errata from last year"
- moved on the sheet: A1, A2, A3, IMU1, J7, J8, U1
